Commit message: Add skarpnack to models. Add script to programatically change model poses

File: resources/urdf/robot_description.xacro (robot description, xacro)
@@ -7,6 +7,5 @@
     <parent link="base_footprint" />
     <child link="base_link" />
-    <!-- Lift it above ground a little bit -->
-    <origin xyz="0 0 0.0501" rpy="0 0 0" />
+    <origin xyz="0 0 0.05" rpy="0 0 0" />
   </joint>
   <link name="base_link">
